File: PCB/CodePad.kicad_pcb (KiCad board)
At the start: 2 copper layers, 24.5 x 66 mm, 9 parts, among them SW1 SW_Push, SW2 SW_Push, SW3 SW_Push, U1 MOUDLE-SEEEDUINO-XIAO

Commit message: Remove unnecessary .DS_Store file from production directory and reogr
Parts:
- added D1: SK6812MINI-E, footprints:SK6812MINI-E_fixed, F.Cu at (3.82, 2.13)
- added D2: SK6812MINI-E, footprints:SK6812MINI-E_fixed, F.Cu at (3.82, 7.18)
- added D3: SK6812MINI-E, footprints:SK6812MINI-E_fixed, F.Cu at (3.82, 12.2)
- added D8: SK6812MINI-E, footprints:SK6812MINI-E_fixed, F.Cu at (3.82, 17.3)
- R1: footprint Resistor_SMD:R_0603_1608Metric_Pad0.98x0.95mm_HandSolder -> Resistor_SMD:R_0603_1608Metric
Connections:
- D6 pad 2: unconnected-(D6-DOUT-Pad2) -> Net-(D6-DOUT)
- D7 pad 2: unconnected-(D7-DOUT-Pad2) -> Net-(D1-DIN)
- D7 pad 4: unconnected-(D7-DIN-Pad4) -> Net-(D6-DOUT)
